File: Digital_Fabrication/Brain/Brain_v10/brain1_v10/brain1_v10.brd (EAGLE design)
At the start: 167.7 x 131.1 mm, 84 parts

Commit message: brain 2 v10!
Parts:
- added J2, J3: (no value), SparkFun-Connectors:1X01_SOLDER_PADS
- moved LED22 3.81 mm to (83.2, 111.0)
- moved J1 3.81 mm to (129.7, 9.64)
- moved LED6 2.54 mm to (118.5, 112.9)
- moved LED62 2.54 mm to (95.2, 50.8)
- moved LED9 2.54 mm to (45.5, 119.8)
- moved LED35 1.27 mm to (55.3, 75.0)
- moved LED41 1.27 mm to (83.2, 85.9)
- moved LED49 1.27 mm to (54.6, 77.5)
- moved LED56 1.27 mm to (90.2, 106.7)
- moved LED71 1.27 mm to (53.8, 123.0)
Connections:
- net GND: now also J2.1, J3.1
Routing:
- net DO: track 0.00 -> 27.2 mm
- net DI: track 0.00 -> 13.6 mm
- net N$35: track 18.3 -> 27.3 mm
- net N$33: track 23.6 -> 31.8 mm
- net N$43: track 19.9 -> 26.4 mm
- net N$58: track 66.9 -> 71.8 mm
- net N$20: track 23.5 -> 19.7 mm
- net N$19: track 26.5 -> 30.3 mm
- net N$72: track 106.8 -> 110.6 mm
- net N$36: track 18.6 -> 21.7 mm
- net N$38: track 34.8 -> 37.7 mm
- net N$76: track 51.9 -> 54.5 mm
- net N$59: track 19.3 -> 16.7 mm
- net N$5: track 22.9 -> 20.4 mm
- net N$10: track 21.4 -> 24.0 mm
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Other:
- board text added: "v10"
