File: Digital_Fabrication/Brain/Brain_v11/brain1_v11/brain1_v11.brd (EAGLE design)
At the start: 167.7 x 131.1 mm, 90 parts, among them J6 ELECTRO_MECH_PAD, J7 ELECTRO_MECH_PAD, J8 ELECTRO_MECH_PAD, J9 ELECTRO_MECH_PAD

Commit message: Add silkscreen
Parts:
- added U$1: FAVICON#SVG, favicon#svg:FAVICON#SVG
- added U$2: BRAIN1_PCB_SILK_1_01_ARTBOARD_1#JPG, Brain1_PCB_silk_1_01_Artboard_1#jpg:BRAIN1_PCB_SILK_1_01_ARTBOARD_1#JPG
Changed lines of the file:
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@@
 <?xml version="1.0" encoding="utf-8"?>
 <!DOCTYPE eagle SYSTEM "eagle.dtd">
-<eagle version="9.5.2">
+<eagle version="9.6.2">
 <drawing>
 <settings>
-<setting alwaysvectorfont="no"/>
+<setting alwaysvectorfont="yes"/>
 <setting verticaltext="up"/>
 </settings>
@@
 <layer number="14" name="Route14" color="1" fill="6" visible="no" active="no"/>
 <layer number="15" name="Route15" color="23" fill="6" visible="no" active="yes"/>
-<layer number="16" name="Bottom" color="1" fill="1" visible="yes" active="yes"/>
+<layer number="16" name="Bottom" color="1" fill="1" visible="no" active="yes"/>
 <layer number="17" name="Pads" color="2" fill="1" visible="yes" active="yes"/>
 <layer number="18" name="Vias" color="2" fill="1" visible="yes" active="yes"/>
@@
 <layer number="20" name="Dimension" color="24" fill="1" visible="yes" active="yes"/>
 <layer number="21" name="tPlace" color="16" fill="1" visible="yes" active="yes"/>
-<layer number="22" name="bPlace" color="14" fill="1" visible="yes" active="yes"/>
+<layer number="22" name="bPlace" color="14" fill="1" visible="no" active="yes"/>
 <layer number="23" name="tOrigins" color="15" fill="1" visible="yes" active="yes"/>
 <layer number="24" name="bOrigins" color="15" fill="1" visible="yes" active="yes"/>
@@
 <layer number="45" name="Holes" color="7" fill="1" visible="yes" active="yes"/>
 <layer number="46" name="Milling" color="3" fill="1" visible="no" active="yes"/>
-<layer number="47" name="Measures" color="7" fill="1" visible="no" active="yes"/>
+<layer number="47" name="Measures" color="7" fill="1" visible="yes" active="yes"/>
 <layer number="48" name="Document" color="7" fill="1" visible="no" active="yes"/>
 <layer number="49" name="Reference" color="7" fill="1" visible="no" active="yes"/>
@@
 <element name="J8" library="brain" package="5X3_SOLDER_PAD" value="ELECTRO_MECH_PAD" x="84.3788" y="51.438759375" smashed="yes" rot="MR270"/>
 <element name="J9" library="brain" package="5X3_SOLDER_PAD" value="ELECTRO_MECH_PAD" x="84.3788" y="102.238759375" smashed="yes" rot="MR90"/>
+<element name="U$1" library="favicon#svg" package="FAVICON#SVG" value="FAVICON#SVG" x="-217.17" y="147.32" smashed="yes"/>
+<element name="U$2" library="Brain1_PCB_silk_1_01_Artboard_1#jpg" package="BRAIN1_PCB_SILK_1_01_ARTBOARD_1#JPG" value="BRAIN1_PCB_SILK_1_01_ARTBOARD_1#JPG" x="83.82" y="67.31" smashed="yes"/>
 </elements>
 <signals>

Commit message: brain boards v11
Added custom silkscreen
Parts:
- added U$10: 5V1, brain:5V1
- added U$11: GND0, brain:GND0
- added U$12: DI0, brain:DI0
- added U$13: DO3, brain:DO3
- added U$14: IN0, buzzard_labels (8):IN0
- added U$15: OUT1, buzzard_labels (8):OUT1
- added U$3: MAKIN_STUFF2, buzzard_labels (5):MAKIN_STUFF2
- added U$4: A_NERVOUS0, buzzard_labels (5):A_NERVOUS0
- added U$5: SYSTEM1, buzzard_labels (5):SYSTEM1
- added U$6: 5V1, buzzard_labels (6):5V1
- added U$7: GND0, buzzard_labels (6):GND0
- added U$8: DO3, buzzard_labels (6):DO3
- added U$9: DI0, buzzard_labels (7):DI0
- U$1: value FAVICON#SVG -> BRAIN1_PCB_BOT_SILK; device favicon#svg:FAVICON#SVG -> brain:BRAIN1_PCB_BOT_SILK
- U$2: value BRAIN1_PCB_SILK_1_01_ARTBOARD_1#JPG -> BRAIN1_PCB_TOP_SILK; device Brain1_PCB_silk_1_01_Artboard_1#jpg:BRAIN1_PCB_SILK_1_01_ARTBOARD_1#JPG -> brain:BRAIN1_PCB_TOP_SILK
- moved U$1 313.0 mm to (85.1, 66.0), flipped to the bottom
- moved U$2 2.54 mm to (83.8, 64.8)
Changed lines of the file:
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@@
 <layers>
 <layer number="1" name="Top" color="4" fill="1" visible="yes" active="yes"/>
-<layer number="2" name="Route2" color="63" fill="3" visible="no" active="yes"/>
+<layer number="2" name="Route2" color="63" fill="3" visible="yes" active="yes"/>
 <layer number="3" name="Route3" color="4" fill="3" visible="no" active="no"/>
 <layer number="4" name="Route4" color="1" fill="4" visible="no" active="no"/>
@@
 <layer number="13" name="Route13" color="4" fill="5" visible="no" active="no"/>
 <layer number="14" name="Route14" color="1" fill="6" visible="no" active="no"/>
-<layer number="15" name="Route15" color="23" fill="6" visible="no" active="yes"/>
-<layer number="16" name="Bottom" color="1" fill="1" visible="no" active="yes"/>
+<layer number="15" name="Route15" color="23" fill="6" visible="yes" active="yes"/>
+<layer number="16" name="Bottom" color="1" fill="1" visible="yes" active="yes"/>
 <layer number="17" name="Pads" color="2" fill="1" visible="yes" active="yes"/>
 <layer number="18" name="Vias" color="2" fill="1" visible="yes" active="yes"/>
@@
 <layer number="20" name="Dimension" color="24" fill="1" visible="yes" active="yes"/>
 <layer number="21" name="tPlace" color="16" fill="1" visible="yes" active="yes"/>
-<layer number="22" name="bPlace" color="14" fill="1" visible="no" active="yes"/>
+<layer number="22" name="bPlace" color="14" fill="1" visible="yes" active="yes"/>
 <layer number="23" name="tOrigins" color="15" fill="1" visible="yes" active="yes"/>
 <layer number="24" name="bOrigins" color="15" fill="1" visible="yes" active="yes"/>
@@
 <layer number="44" name="Drills" color="7" fill="1" visible="no" active="yes"/>
 <layer number="45" name="Holes" color="7" fill="1" visible="yes" active="yes"/>
-<layer number="46" name="Milling" color="3" fill="1" visible="no" active="yes"/>
-<layer number="47" name="Measures" color="7" fill="1" visible="yes" active="yes"/>
+<layer number="46" name="Milling" color="3" fill="1" visible="yes" active="yes"/>
+<layer number="47" name="Measures" color="7" fill="1" visible="no" active="yes"/>
 <layer number="48" name="Document" color="7" fill="1" visible="no" active="yes"/>
 <layer number="49" name="Reference" color="7" fill="1" visible="no" active="yes"/>
@@
 <element name="J8" library="brain" package="5X3_SOLDER_PAD" value="ELECTRO_MECH_PAD" x="84.3788" y="51.438759375" smashed="yes" rot="MR270"/>
 <element name="J9" library="brain" package="5X3_SOLDER_PAD" value="ELECTRO_MECH_PAD" x="84.3788" y="102.238759375" smashed="yes" rot="MR90"/>
-<element name="U$1" library="favicon#svg" package="FAVICON#SVG" value="FAVICON#SVG" x="-217.17" y="147.32" smashed="yes"/>
-<element name="U$2" library="Brain1_PCB_silk_1_01_Artboard_1#jpg" package="BRAIN1_PCB_SILK_1_01_ARTBOARD_1#JPG" value="BRAIN1_PCB_SILK_1_01_ARTBOARD_1#JPG" x="83.82" y="67.31" smashed="yes"/>
+<element name="U$2" library="brain" package="BRAIN1_PCB_TOP_SILK" value="BRAIN1_PCB_TOP_SILK" x="83.82" y="64.77" smashed="yes"/>
+<element name="U$1" library="brain" package="BRAIN1_PCB_BOT_SILK" value="BRAIN1_PCB_BOT_SILK" x="85.09" y="66.04" smashed="yes" rot="MR0"/>
+<element name="U$3" library="buzzard_labels (5)" package="MAKIN_STUFF2" value="MAKIN_STUFF2" x="121.92" y="11.43" smashed="yes" rot="MR0"/>
+<element name="U$4" library="buzzard_labels (5)" package="A_NERVOUS0" value="A_NERVOUS0" x="100.33" y="13.97" smashed="yes"/>
+<element name="U$5" library="buzzard_labels (5)" package="SYSTEM1" value="SYSTEM1" x="102.87" y="10.16" smashed="yes"/>
+<element name="U$6" library="buzzard_labels (6)" package="5V1" value="5V1" x="133.35" y="5.334" smashed="yes" rot="R90"/>
+<element name="U$7" library="buzzard_labels (6)" package="GND0" value="GND0" x="135.89" y="5.334" smashed="yes" rot="R90"/>
+<element name="U$8" library="buzzard_labels (6)" package="DO3" value="DO3" x="128.27" y="5.334" smashed="yes" rot="R90"/>
+<element name="U$9" library="buzzard_labels (7)" package="DI0" value="DI0" x="130.81" y="5.334" smashed="yes" rot="R90"/>
+<element name="U$10" library="brain" package="5V1" value="5V1" x="133.35" y="5.334" smashed="yes" rot="MR90"/>
+<element name="U$11" library="brain" package="GND0" value="GND0" x="135.89" y="5.334" smashed="yes" rot="MR90"/>
+<element name="U$12" library="brain" package="DI0" value="DI0" x="130.81" y="5.334" smashed="yes" rot="MR90"/>
+<element name="U$13" library="brain" package="DO3" value="DO3" x="128.27" y="5.334" smashed="yes" rot="MR90"/>
+<element name="U$14" library="buzzard_labels (8)" package="IN0" value="IN0" x="132.969" y="15.113" smashed="yes"/>
+<element name="U$15" library="buzzard_labels (8)" package="OUT1" value="OUT1" x="139.319" y="15.24" smashed="yes" rot="MR0"/>
 </elements>
 <signals>
@@
 <contactref element="LED2" pad="4"/>
 <contactref element="LED1" pad="4"/>
-<polygon width="0.025" layer="1">
+<polygon width="0.1524" layer="1">
 <vertex x="0" y="0"/>
 <vertex x="0" y="132.08"/>
@@
 <contactref element="LED39" pad="4"/>
 <contactref element="LED40" pad="4"/>
-<wire x1="138.845" y1="22.69" x2="138.8704" y2="22.6646" width="0.254" layer="1"/>
-<wire x1="18.125" y1="65.9" x2="18.0594" y2="65.9656" width="0.254" layer="1"/>
-<wire x1="29.24" y1="73.305" x2="29.0616" y2="73.1266" width="0.254" layer="1"/>
-<wire x1="117.875" y1="79.1" x2="117.9322" y2="79.0428" width="0.254" layer="1"/>
 <contactref element="LED45" pad="4"/>
 <contactref element="LED44" pad="4"/>
@@
 <contactref element="J5" pad="3"/>
 <wire x1="137.095" y1="22.24" x2="137.095" y2="20.193" width="0.254" layer="1"/>
-<wire x1="137.922" y1="20.193" x2="138.43" y2="20.193" width="0.254" layer="1"/>
-<wire x1="138.43" y1="20.193" x2="142.24" y2="20.193" width="0.254" layer="1"/>
+<wire x1="137.095" y1="20.193" x2="142.24" y2="20.193" width="0.254" layer="1"/>
 <wire x1="142.24" y1="20.193" x2="142.74" y2="19.693" width="0.254" layer="1"/>
 <wire x1="142.74" y1="19.693" x2="142.74" y2="17.78" width="0.254" layer="1"/>
@@
 <wire x1="132.588" y1="20.193" x2="137.095" y2="20.193" width="0.254" layer="1"/>
 <wire x1="130.81" y1="18.415" x2="132.588" y2="20.193" width="0.254" layer="1"/>
-<wire x1="137.922" y1="20.193" x2="137.095" y2="20.193" width="0.254" layer="1"/>
 </signal>
 <signal name="DO">
