File: Digital_Fabrication/Brain/Brain_v11/brain2_v11/brain2_v11.sch (EAGLE design)
At the start: 90 parts, among them J6 ELECTRO_MECH_PAD, J7 ELECTRO_MECH_PAD, J8 ELECTRO_MECH_PAD, J9 ELECTRO_MECH_PAD

Commit message: brain boards v11
Added custom silkscreen
Parts:
- added U$1: A_NERVOUS0, brain:A_NERVOUS0
- added U$10, U$11: DO3, brain:DO3
- added U$12: IN0, brain:IN0
- added U$13: OUT1, brain:OUT1
- added U$14: BRAIN2_PCB_TOP_SILK, brain:BRAIN2_PCB_TOP_SILK
- added U$15: BRAIN2_PCB_BOT_SILK, brain:BRAIN2_PCB_BOT_SILK
- added U$2: SYSTEM1, brain:SYSTEM1
- added U$3: MAKIN_STUFF2, brain:MAKIN_STUFF2
- added U$4, U$5: 5V1, brain:5V1
- added U$6, U$7: GND0, brain:GND0
- added U$8, U$9: DI0, brain:DI0
Other:
- note added: "Aesthetics"
Changed lines of the file:
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@@
 <?xml version="1.0" encoding="utf-8"?>
 <!DOCTYPE eagle SYSTEM "eagle.dtd">
-<eagle version="9.5.2">
+<eagle version="9.6.2">
 <drawing>
 <settings>
@@
 <part name="J8" library="brain" deviceset="ELECTRO_MECH_PAD" device=""/>
 <part name="J9" library="brain" deviceset="ELECTRO_MECH_PAD" device=""/>
+<part name="U$1" library="brain" deviceset="A_NERVOUS0" device=""/>
+<part name="U$2" library="brain" deviceset="SYSTEM1" device=""/>
+<part name="U$3" library="brain" deviceset="MAKIN_STUFF2" device=""/>
+<part name="U$4" library="brain" deviceset="5V1" device=""/>
+<part name="U$5" library="brain" deviceset="5V1" device=""/>
+<part name="U$6" library="brain" deviceset="GND0" device=""/>
+<part name="U$7" library="brain" deviceset="GND0" device=""/>
+<part name="U$8" library="brain" deviceset="DI0" device=""/>
+<part name="U$9" library="brain" deviceset="DI0" device=""/>
+<part name="U$10" library="brain" deviceset="DO3" device=""/>
+<part name="U$11" library="brain" deviceset="DO3" device=""/>
+<part name="U$12" library="brain" deviceset="IN0" device=""/>
+<part name="U$13" library="brain" deviceset="OUT1" device=""/>
+<part name="U$14" library="brain" deviceset="BRAIN2_PCB_TOP_SILK" device=""/>
+<part name="U$15" library="brain" deviceset="BRAIN2_PCB_BOT_SILK" device=""/>
 </parts>
 <sheets>
@@
 <text x="7.62" y="190.5" size="2.54" layer="97" font="vector">Headers</text>
 <text x="7.62" y="144.78" size="2.54" layer="97" font="vector">Electro-mechanical pads</text>
+<text x="5.08" y="25.4" size="2.54" layer="97" font="vector">Aesthetics</text>
 </plain>
 <instances>
@@
 <attribute name="NAME" x="7.62" y="86.868" size="1.778" layer="95" font="vector"/>
 </instance>
+<instance part="U$1" gate="G$1" x="38.1" y="15.24" smashed="yes"/>
+<instance part="U$2" gate="G$1" x="38.1" y="10.16" smashed="yes"/>
+<instance part="U$3" gate="G$1" x="38.1" y="5.08" smashed="yes"/>
+<instance part="U$4" gate="G$1" x="58.42" y="20.32" smashed="yes"/>
+<instance part="U$5" gate="G$1" x="66.04" y="20.32" smashed="yes"/>
+<instance part="U$6" gate="G$1" x="58.42" y="15.24" smashed="yes"/>
+<instance part="U$7" gate="G$1" x="66.04" y="15.24" smashed="yes"/>
+<instance part="U$8" gate="G$1" x="58.42" y="10.16" smashed="yes"/>
+<instance part="U$9" gate="G$1" x="66.04" y="10.16" smashed="yes"/>
+<instance part="U$10" gate="G$1" x="58.42" y="5.08" smashed="yes"/>
+<instance part="U$11" gate="G$1" x="66.04" y="5.08" smashed="yes"/>
+<instance part="U$12" gate="G$1" x="76.2" y="10.16" smashed="yes"/>
+<instance part="U$13" gate="G$1" x="76.2" y="5.08" smashed="yes"/>
+<instance part="U$14" gate="G$1" x="5.08" y="10.16" smashed="yes"/>
+<instance part="U$15" gate="G$1" x="5.08" y="5.08" smashed="yes"/>
 </instances>
 <busses>
